File: hardware/vga_breakout.brd (EAGLE design)
At the start: 27.9 x 49.8 mm, 11 parts, among them J1 VGA_DB15, J2 HEADER_5P

Commit message: added +5V line to breakout PCB
Parts:
- removed J2: HEADER_5P, mw-voice-marker:HEADER_5P
- added U$9: HEADER_6P, mw-voice-marker:HEADER_6P
Connections:
- new net +5V: J1.9, U$9.1
- net GND: now also U$9.6; no longer J2.5
- net HSYNC: now also U$9.2; no longer J2.1
- net SCL: now also U$9.5; no longer J2.4
- net SDA: now also U$9.4; no longer J2.3
- net VSYNC: now also U$9.3; no longer J2.2
Routing:
- net +5V: track 0.00 -> 43.5 mm, vias 0 -> 6
- net VSYNC: track 32.5 -> 34.7 mm
- net SCL: track 41.3 -> 43.0 mm
Other:
- board text added: "+5V"
Changed lines of the file:
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@@
 <text x="20.6375" y="11.1125" size="1.4224" layer="21" ratio="12" rot="R90">Blue</text>
 <text x="20.6375" y="41.5925" size="1.4224" layer="21" ratio="12" rot="R90">Red</text>
-<text x="14.605" y="44.1325" size="1.4224" layer="21" ratio="12" rot="R270">GND</text>
-<text x="12.065" y="44.1325" size="1.4224" layer="21" ratio="12" rot="R270">SCL</text>
-<text x="9.525" y="44.1325" size="1.4224" layer="21" ratio="12" rot="R270">SDA</text>
-<text x="6.985" y="44.1325" size="1.4224" layer="21" ratio="12" rot="R270">VS</text>
-<text x="4.445" y="44.1325" size="1.4224" layer="21" ratio="12" rot="R270">HS</text>
+<text x="16.1925" y="44.45" size="1.4224" layer="21" ratio="12" rot="R270">GND</text>
+<text x="13.6525" y="44.45" size="1.4224" layer="21" ratio="12" rot="R270">SCL</text>
+<text x="10.795" y="44.45" size="1.4224" layer="21" ratio="12" rot="R270">SDA</text>
+<text x="8.255" y="44.45" size="1.4224" layer="21" ratio="12" rot="R270">VS</text>
+<text x="5.715" y="44.45" size="1.4224" layer="21" ratio="12" rot="R270">HS</text>
+<text x="3.175" y="44.45" size="1.4224" layer="21" ratio="12" rot="R270">+5V</text>
 </plain>
 <attributes>
@@
 <element name="R5" library="mw-voice-marker" package="R0805" value="43.2" x="19.05" y="9.525" rot="R180"/>
 <element name="R6" library="mw-voice-marker" package="R0805" value="86.6" x="19.05" y="6.985" rot="R180"/>
-<element name="J2" library="mw-voice-marker" package="HEADER_5P" value="HEADER_5P" x="10.16" y="45.72"/>
+<element name="U$9" library="mw-voice-marker" package="HEADER_6P" value="HEADER_6P" x="10.16" y="46.355"/>
 </elements>
 <signals>
@@
 <vertex x="0" y="50.165"/>
 </polygon>
-<contactref element="J2" pad="5"/>
 <via x="1.27" y="1.27" extent="1-16" drill="0.55"/>
 <via x="5.08" y="1.27" extent="1-16" drill="0.55"/>
@@
 <via x="16.51" y="40.005" extent="1-16" drill="0.3"/>
 <via x="18.0975" y="35.8775" extent="1-16" drill="0.3"/>
+<contactref element="U$9" pad="6"/>
 </signal>
 <signal name="SDA">
 <contactref element="J1" pad="12"/>
-<contactref element="J2" pad="3"/>
-<wire x1="10.16" y1="45.72" x2="6.0325" y2="41.5925" width="0.4064" layer="1"/>
-<wire x1="6.0325" y1="41.5925" x2="6.0325" y2="28.2575" width="0.4064" layer="1"/>
-<wire x1="6.0325" y1="28.2575" x2="7.485" y2="26.805" width="0.4064" layer="1"/>
-<wire x1="7.485" y1="26.805" x2="8.89" y2="26.805" width="0.4064" layer="1"/>
+<contactref element="U$9" pad="4"/>
+<wire x1="11.43" y1="46.355" x2="11.43" y2="43.4975" width="0.3048" layer="1"/>
+<wire x1="11.43" y1="43.4975" x2="7.9375" y2="40.005" width="0.3048" layer="1"/>
+<wire x1="7.9375" y1="40.005" x2="7.9375" y2="33.655" width="0.3048" layer="1"/>
+<wire x1="7.9375" y1="33.655" x2="10.16" y2="31.4325" width="0.3048" layer="1"/>
+<wire x1="10.16" y1="31.4325" x2="10.16" y2="28.075" width="0.3048" layer="1"/>
+<wire x1="10.16" y1="28.075" x2="8.89" y2="26.805" width="0.3048" layer="1"/>
 </signal>
 <signal name="SCL">
 <contactref element="J1" pad="15"/>
-<contactref element="J2" pad="4"/>
-<wire x1="12.7" y1="45.72" x2="10.4775" y2="47.9425" width="0.4064" layer="1"/>
-<wire x1="2.9337" y1="46.90396875" x2="2.9337" y2="24.6888" width="0.4064" layer="1"/>
-<wire x1="7.6875" y1="19.935" x2="8.89" y2="19.935" width="0.4064" layer="1"/>
-<wire x1="2.9337" y1="24.6888" x2="7.6875" y2="19.935" width="0.4064" layer="1"/>
-<wire x1="3.97223125" y1="47.9425" x2="2.9337" y2="46.90396875" width="0.4064" layer="1"/>
-<wire x1="10.4775" y1="47.9425" x2="3.97223125" y2="47.9425" width="0.4064" layer="1"/>
+<contactref element="U$9" pad="5"/>
+<wire x1="2.98561875" y1="48.0822" x2="2.0828" y2="47.17938125" width="0.3048" layer="1"/>
+<wire x1="2.0828" y1="47.17938125" x2="2.0828" y2="45.21311875" width="0.3048" layer="1"/>
+<wire x1="2.0828" y1="45.21311875" x2="3.81" y2="43.48591875" width="0.3048" layer="1"/>
+<wire x1="13.97" y1="46.355" x2="13.36395" y2="46.355" width="0.3048" layer="1"/>
+<wire x1="13.36395" y1="46.355" x2="11.63675" y2="48.0822" width="0.3048" layer="1"/>
+<wire x1="11.63675" y1="48.0822" x2="2.98561875" y2="48.0822" width="0.3048" layer="1"/>
+<wire x1="3.81" y1="26.035" x2="7.3025" y2="22.5425" width="0.3048" layer="1"/>
+<wire x1="7.3025" y1="22.5425" x2="7.3025" y2="21.5225" width="0.3048" layer="1"/>
+<wire x1="7.3025" y1="21.5225" x2="8.89" y2="19.935" width="0.3048" layer="1"/>
+<wire x1="3.81" y1="43.48591875" x2="3.81" y2="26.035" width="0.3048" layer="1"/>
 </signal>
 <signal name="N$1">
@@
 </signal>
 <signal name="VSYNC">
-<contactref element="J2" pad="2"/>
 <contactref element="J1" pad="14"/>
-<wire x1="7.62" y1="45.72" x2="6.0325" y2="47.3075" width="0.4064" layer="1"/>
-<wire x1="6.0325" y1="47.3075" x2="4.1275" y2="47.3075" width="0.4064" layer="1"/>
-<wire x1="4.1275" y1="47.3075" x2="3.4925" y2="46.6725" width="0.4064" layer="1"/>
-<wire x1="3.4925" y1="43.18" x2="4.1275" y2="42.545" width="0.4064" layer="1"/>
-<wire x1="4.1275" y1="42.545" x2="4.1275" y2="25.7175" width="0.4064" layer="1"/>
-<wire x1="4.1275" y1="25.7175" x2="7.62" y2="22.225" width="0.4064" layer="1"/>
-<wire x1="7.62" y1="22.225" x2="8.89" y2="22.225" width="0.4064" layer="1"/>
-<wire x1="3.4925" y1="46.6725" x2="3.4925" y2="43.18" width="0.4064" layer="1"/>
+<contactref element="U$9" pad="3"/>
+<wire x1="8.89" y1="46.355" x2="7.62" y2="47.625" width="0.3048" layer="1"/>
+<wire x1="7.62" y1="47.625" x2="3.175" y2="47.625" width="0.3048" layer="1"/>
+<wire x1="3.175" y1="47.625" x2="2.54" y2="46.99" width="0.3048" layer="1"/>
+<wire x1="2.54" y1="46.99" x2="2.54" y2="45.4025" width="0.3048" layer="1"/>
+<wire x1="2.54" y1="45.4025" x2="4.445" y2="43.4975" width="0.3048" layer="1"/>
+<wire x1="4.445" y1="43.4975" x2="4.445" y2="26.3525" width="0.3048" layer="1"/>
+<wire x1="4.445" y1="26.3525" x2="8.5725" y2="22.225" width="0.3048" layer="1"/>
+<wire x1="8.5725" y1="22.225" x2="8.89" y2="22.225" width="0.3048" layer="1"/>
 </signal>
 <signal name="HSYNC">
 <contactref element="J1" pad="13"/>
-<contactref element="J2" pad="1"/>
-<wire x1="5.08" y1="45.72" x2="5.08" y2="27.305" width="0.4064" layer="1"/>
-<wire x1="7.87" y1="24.515" x2="8.89" y2="24.515" width="0.4064" layer="1"/>
-<wire x1="5.08" y1="27.305" x2="7.87" y2="24.515" width="0.4064" layer="1"/>
+<contactref element="U$9" pad="2"/>
+<wire x1="8.89" y1="24.515" x2="7.3025" y2="26.1025" width="0.3048" layer="1"/>
+<wire x1="7.3025" y1="45.4025" x2="6.35" y2="46.355" width="0.3048" layer="1"/>
+<wire x1="7.3025" y1="26.1025" x2="7.3025" y2="45.4025" width="0.3048" layer="1"/>
+</signal>
+<signal name="+5V">
+<contactref element="U$9" pad="1"/>
+<contactref element="J1" pad="9"/>
+<wire x1="11.43" y1="23.37" x2="10.16" y2="22.1" width="0.3048" layer="1"/>
+<wire x1="10.16" y1="22.1" x2="10.16" y2="18.415" width="0.3048" layer="1"/>
+<wire x1="10.16" y1="18.415" x2="6.0325" y2="18.415" width="0.6096" layer="1"/>
+<via x="6.0325" y="18.415" extent="1-16" drill="0.6"/>
+<wire x1="6.0325" y1="18.415" x2="6.0325" y2="28.8925" width="0.6096" layer="16"/>
+<via x="6.0325" y="28.8925" extent="1-16" drill="0.6"/>
+<wire x1="6.0325" y1="28.8925" x2="6.0325" y2="30.1625" width="0.6096" layer="1"/>
+<wire x1="6.0325" y1="31.4325" x2="6.0325" y2="44.1325" width="0.6096" layer="1"/>
+<wire x1="6.0325" y1="44.1325" x2="3.81" y2="46.355" width="0.6096" layer="1"/>
+<via x="6.0325" y="30.1625" extent="1-16" drill="0.6"/>
+<via x="6.0325" y="31.4325" extent="1-16" drill="0.6"/>
+<via x="6.0325" y="19.685" extent="1-16" drill="0.6"/>
+<via x="6.0325" y="20.955" extent="1-16" drill="0.6"/>
+<wire x1="6.0325" y1="18.415" x2="6.0325" y2="19.685" width="0.6096" layer="1"/>
+<wire x1="6.0325" y1="28.8925" x2="6.0325" y2="31.4325" width="0.6096" layer="16"/>
+<wire x1="6.0325" y1="31.4325" x2="6.0325" y2="30.1625" width="0.6096" layer="1"/>
+<wire x1="6.0325" y1="20.955" x2="6.0325" y2="19.685" width="0.6096" layer="1"/>
 </signal>
 </signals>
